Commit message: mesh file cleanup and minor changes

File: urdf/head.urdf (robot description, URDF)
Before this commit: robot urdf-head, 7 links, 6 joints
Links:
- link base_link: geometry visual mesh filename=../meshes/base_link.STL
- link chin: geometry visual mesh filename=../meshes/chin.STL
- link d455_link: geometry visual mesh filename=../meshes/d455_link.STL
- link face: geometry visual mesh filename=../meshes/face.STL
- link mid360_link: geometry visual mesh filename=../meshes/mid360_link.STL
- link neck: geometry visual mesh filename=../meshes/neck.STL
